Commit message: Add visual representation for wheel links

File: Model/car_object.urdf (robot description, URDF)
Before this commit: robot car, 8 links, 5 joints
Links:
- removed link bl_wheel_to_drive_axle
- added link bl_wheel; visual cylinder length=1 radius=2
- link br_wheel: geometry visual cylinder length=1 radius=2
- link fl_wheel: geometry visual cylinder length=1 radius=2
- link fr_wheel: geometry visual cylinder length=1 radius=2

Commit message: Add visual elements to car model components

File: Model/car_object.urdf (robot description, URDF)
Before this commit: robot car, 8 links, 5 joints
Links:
- link body: geometry visual box size=6 2 2
- link drive_axle: geometry visual cylinder length=6 radius=0.1
- link steer_axle: geometry visual cylinder length=6 radius=0.1

Commit message: Update car_object.urdf

File: Model/car_object.urdf (robot description, URDF)
Before this commit: robot car, 8 links, 5 joints
Joints:
- added joint bl_wheel_to_drive_axle: type continuous, parent , child 
- joint br_wheel_to_drive_axle: child (none) -> ; parent (none) -> ; type None -> continuous
- joint drive_axle_to_car: child (none) -> ; parent (none) -> ; type None -> continuous
- joint fl_wheel_to_steer_axle: child (none) -> ; parent (none) -> ; type None -> continuous
- joint fr_wheel_to_steer_axle: child (none) -> ; parent (none) -> ; type None -> continuous
- joint steer_axle_to_car: child (none) -> ; parent (none) -> ; type None -> continuous

Commit message: Update car_object.urdf

File: Model/car_object.urdf (robot description, URDF)
Before this commit: robot car, 8 links, 6 joints
Joints:
- added joint fl_wheel_to_steer_pivot: type prismatic, parent steer_pivot, child fl_wheel
- added joint fr_wheel_to_steer_pivot: type prismatic, parent steer_pivot, child fr_wheel
- added joint steer_pivot_to_car: type prismatic, parent body, child steer_pivot
- joint bl_wheel_to_drive_axle: child  -> bl_wheel; parent  -> drive_axle
- joint br_wheel_to_drive_axle: child  -> br_wheel; parent  -> drive_axle
- joint drive_axle_to_car: child  -> drive_axle; parent  -> body
- joint fl_wheel_to_steer_axle: child  -> fl_wheel; parent  -> steer_axle
- joint fr_wheel_to_steer_axle: child  -> fr_wheel; parent  -> steer_axle
- joint steer_axle_to_car: child  -> steer_axle; parent  -> body
